File: warps/hardware_design/pcb/kicad/warps.kicad_pcb (KiCad board)
At the start: 2 copper layers, 48.9 x 106.7 mm, 126 parts, among them IC1 LM1117-3.3, IC2 LM4040B10, IC3 MCP6004, IC4 STM32F405RGT6, IC5 WM8731, IC6 TL072, J1 PJ301_THONKICONN6, J2 PJ301_THONKICONN6, J3 PJ301_THONKICONN6, J4 PJ301_THONKICONN6, J5 PJ301_THONKICONN6, J6 PJ301_THONKICONN6, J7 PJ301_THONKICONN6, J8 PJ301_THONKICONN6, Q1 8MHz, Q2 12.288MHz, SW1 EVQQ2, SW2 EVQQ2, SW3 TAC_SWITCHPTH

Commit message: warps extra via
Routing:
- net GND: vias 60 -> 61
Changed lines of the file:
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@@
   (via (at 158.1 123) (size 1.108) (drill 0.6) (layers "F.Cu" "B.Cu") (net 1))
   (via (at 134.8486 58.9661) (size 1.108) (drill 0.6) (layers "F.Cu" "B.Cu") (net 1))
+  (via (at 152 92) (size 1.108) (drill 0.6) (layers "F.Cu" "B.Cu") (net 1))
   (via (at 167.1 121.9) (size 1.108) (drill 0.6) (layers "F.Cu" "B.Cu") (net 1))
   (via (at 171.3611 62.1411) (size 1.108) (drill 0.6) (layers "F.Cu" "B.Cu") (net 1))
