File: tides2/hardware_design/pcb/kicad/tides_2.kicad_sch (KiCad schematic)
At the start: 20 parts

Commit message: tides final tweaks
Parts:
- C1, C12, C13, C16: value (none) -> 1u; footprint (none) -> tides:C0402
- C11, C4: value (none) -> 20p; footprint (none) -> tides:C0402
- C14, C15, C2, C3, C8: value (none) -> 100n; footprint (none) -> tides:C0402
- IC1: value (none) -> STM32F373CCT6; footprint (none) -> tides:LQFP48
- JP6: value (none) -> M04PTH; footprint (none) -> tides:1X04
- JP7: value (none) -> M02PTH; footprint (none) -> tides:1X02
- Q1: value (none) -> 8MHz; footprint (none) -> tides:CTS406
- R3: value (none) -> 10k; footprint (none) -> tides:R0402
- R4, R5, R8, R9: value (none) -> 100; footprint (none) -> tides:R0402
