File: tides2/hardware_design/pcb/kicad/tides_3.kicad_sch (KiCad schematic)
At the start: 39 parts

Commit message: tides final tweaks
Parts:
- C22, C23, C35, C44, C45, C5, C51, C52, C53, C54, C55: value (none) -> 100n; footprint (none) -> tides:C0402
- C56: value (none) -> 1.0n; footprint (none) -> tides:C0402
- IC2: value (none) -> 4051PW; footprint (none) -> tides:TSSOP16_065
- JP1, JP2, JP3, JP4: value (none) -> FIDUCIAL1X2; footprint (none) -> tides:FIDUCIAL-1X2
- LED1, LED2, LED3: value (none) -> W115WSURKMGKW; footprint (none) -> tides:LED-BICOLOR-THROUGHHOLE-2.54
- R1, R13, R7: value (none) -> 2.4k; footprint (none) -> tides:R0402
- R10, R2, R6: value (none) -> 1.5k; footprint (none) -> tides:R0402
- R11, R12, R22, R23, R24: value (none) -> 10kB; footprint (none) -> tides:ALPS_POT_VERTICAL_PS
- R56, R57, R58, R59, R60: value (none) -> 10kB; footprint (none) -> tides:ALPS_POT_VERTICAL
- SW1, SW2, SW3: value (none) -> TAC_SWITCHPTH; footprint (none) -> tides:TACTILE-PTH
