File: tides2/hardware_design/pcb/kicad/tides_4.kicad_sch (KiCad schematic)
At the start: 56 parts

Commit message: tides final tweaks
Parts:
- C27, C31, C36: value (none) -> 100p; footprint (none) -> tides:C0402
- C28, C32, C41, C46, C47: value (none) -> 1.0n; footprint (none) -> tides:C0402
- C30, C43: value (none) -> 100n; footprint (none) -> tides:C0402
- D10, D11, D4, D5, D6, D7, D8, D9: value (none) -> TVS; footprint (none) -> tides:0603
- D2: value (none) -> BAT54S; footprint (none) -> tides:SOT23
- IC6, IC7: value (none) -> MCP6004; footprint (none) -> tides:TSSOP14_065
- J1, J2, J3, J4, J5, J6, J7, J8: value (none) -> PJ301_THONKICONN6; footprint (none) -> tides:WQP_PJ_301M6
- R16, R17, R29, R30, R35, R36, R54, R55: value (none) -> 100k; footprint (none) -> tides:R0402
- R18, R19, R27, R41, R52: value (none) -> 20k; footprint (none) -> tides:R0402
- R20, R21, R25, R43, R51: value (none) -> 120k; footprint (none) -> tides:R0402
- R26, R44: value (none) -> 390k; footprint (none) -> tides:R0402
- R28, R37: value (none) -> 130k; footprint (none) -> tides:R0402
- R50: value (none) -> 140k; footprint (none) -> tides:R0402
- R53: value (none) -> 33k; footprint (none) -> tides:R0402
- R61, R62, R63: value (none) -> 10k; footprint (none) -> tides:R0402
