File: tides2/hardware_design/pcb/kicad/tides_6.kicad_sch (KiCad schematic)
At the start: 21 parts

Commit message: tides final tweaks
Parts:
- C10, C50, C9: value (none) -> 10u; footprint (none) -> tides:PANASONIC_B
- C19, C20, C25: value (none) -> 22u; footprint (none) -> tides:C1206
- C24, C26: value (none) -> 22u; footprint (none) -> tides:PANASONIC_B
- C42: value (none) -> 1u; footprint (none) -> tides:C0402
- C7: value (none) -> 100n; footprint (none) -> tides:C0402
- D1, D3: value (none) -> 1N5819HW; footprint (none) -> tides:SOD123
- IC10: value (none) -> LM4040B10; footprint (none) -> tides:DBZ_R-PDSO-G3
- IC3: value (none) -> R-78E3.3-0.5; footprint (none) -> tides:WE78
- IC5: value (none) -> LD2981ABU33; footprint (none) -> tides:SOT89
- JP5: value (none) -> M05X2SHD; footprint (none) -> tides:2X5-SHROUDED
- L1: value (none) -> 33u; footprint (none) -> tides:L2012C
- L2, L3, L4: value (none) -> WE-CBF_0603; footprint (none) -> tides:0603
- R46: value (none) -> 1.5k; footprint (none) -> tides:R0402
