File: marbles/hardware_design/pcb/kicad/marbles.kicad_pcb (KiCad board)
At the start: 2 copper layers, 88.9 x 106 mm, 211 parts, among them IC1 R-78E3.3-0.5, IC10 TL074PW, IC2 STM32F405RGT6, IC3 LD2981ABU33, IC4 DAC8565, IC5 MCP6004, IC6 MCP6004, IC7 OPA4171, IC8 LM4040B10, IC9 LM324PW, J1 PJ301_THONKICONN6, J10 PJ301_THONKICONN6, J11 PJ301_THONKICONN6, J12 PJ301_THONKICONN6, J13 PJ301_THONKICONN6, J14 PJ301_THONKICONN6, J15 PJ301_THONKICONN6, J16 PJ301_THONKICONN6, J17 Conn_01x04_Male, J2 PJ301_THONKICONN6, J3 PJ301_THONKICONN6, J4 PJ301_THONKICONN6, J5 PJ301_THONKICONN6, J6 PJ301_THONKICONN6, J7 PJ301_THONKICONN6, J8 PJ301_THONKICONN6, J9 PJ301_THONKICONN6, Q1 8MHz, Q2 MMBT3904, Q3 MMBT3904, SW1 SW_Push_LED, SW2 SW_Push_LED, SW3 TAC_SWITCHPTH, SW4 TAC_SWITCHPTH, SW5 TAC_SWITCHPTH, SW6 TAC_SWITCHPTH, SW7 TAC_SWITCHPTH

Commit message: marbles change button LEDs from 1k to 680R
Parts:
- R1, R5: value 1k -> 680

Commit message: marbles silkscreen for calibration readings
Other:
- board text added: "y1, y3: x11, x13: x21, x23: x31, x33:"
Changed lines of the file:
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@@
     (effects (font (size 0.92837 0.92837) (thickness 0.16383)) (justify left bottom mirror))
+  )
+  (gr_text "y1, y3:                                 \n\nx11, x13:\n\nx21, x23:\n\nx31, x33:\n\n\n " (at 163.7 88.7) (layer "B.SilkS" knockout)
+    (effects (font (size 1 1) (thickness 0.15)) (justify left bottom mirror))
   )
   (gr_text "GND" (at 136.4361 62.4586 -90) (layer "B.SilkS")

Commit message: marbles rotate output LEDs to match original
Parts:
- turned LED10 to 180 degrees
- turned LED11 to 180 degrees
- turned LED12 to 180 degrees
- turned LED6 to 180 degrees
- turned LED7 to 180 degrees
- turned LED8 to 180 degrees
- turned LED9 to 180 degrees
Routing:
- net Net-(IC10A--IN): track 28.2 -> 25.1 mm
- net Net-(IC10C-OUT): track 42.7 -> 45.2 mm
- net Net-(IC10B--IN): track 30.7 -> 28.2 mm
- net Net-(IC10A-OUT): track 21.3 -> 23.1 mm
- net Net-(IC10D-OUT): track 32.4 -> 34.2 mm
- net Net-(IC10B-OUT): track 23.2 -> 21.8 mm, vias 1 -> 0
- net GATE_T_3: track 82.1 -> 80.8 mm
- net Net-(IC9C-OUT): track 43.1 -> 42.0 mm
- net GATE_T_2: track 95.9 -> 95.0 mm
- net Net-(IC10C--IN): track 30.9 -> 30.2 mm
